Commit message: [FEAT]  Add Kinect

File: catkin_ws/src/robot/urdf/my_robot.xacro (robot description, xacro)
@@ -2,5 +2,5 @@
 <robot name="my_robot" xmlns:xacro="http://www.ros.org/wiki/xacro">
 	<include filename="$(find robot)/urdf/my_robot.gazebo" />
-	<!--  Footprint -->
+	<!-- Footprint -->
 	<link name="robot_footprint">
 	</link>
@@ -175,5 +175,5 @@
 			<origin xyz="-0.0 0 0" rpy=" 0 0 0" />
 			<geometry>
-				<box size="0.05 0.05 0.05" />
+				<mesh filename="package://robot/meshes/kinect.dae" />
 			</geometry>
 		</visual>
@@ -196,9 +196,4 @@
 		<axis xyz="0 1 0" rpy="0 0 0" />
 	</joint>
-	<gazebo reference="camera">
-		<material>
-			Gazebo/Red
-		</material>
-	</gazebo>
 	<!-- LIDAR -->
 	<link name="hokuyo">

Commit message: [FIX] Update depth camera frame

File: catkin_ws/src/robot/urdf/my_robot.xacro (robot description, xacro)
@@ -173,5 +173,30 @@
 	<link name="camera">
 		<visual>
-			<origin xyz="-0.0 0 0" rpy=" 0 0 0" />
+			<origin xyz="-0.0 0 0.0" rpy=" 0 0 0" />
+			<geometry>
+				<box size="0.05 0.05 0.05" />
+			</geometry>
+		</visual>
+		<collision>
+			<origin xyz="-0.0 0 0" rpy=" 0 0 0" />
+			<geometry>
+				<box size="0.05 0.05 0.05" />
+			</geometry>
+		</collision>
+		<inertial>
+			<mass value="0.1" />
+			<origin xyz="0.0 0 0" rpy=" 0 0 0" />
+			<inertia ixx="1e-6" ixy="0" ixz="0" iyy="1e-6" iyz="0" izz="1e-6" />
+		</inertial>
+	</link>
+	<joint type="fixed" name="camera_joint">
+		<origin xyz="0.4 0 0.0" rpy="0 0 0" />
+		<child link="camera" />
+		<parent link="chassis" />
+	</joint>
+	<!-- RGBD Camera -->
+	<link name="RGBD_camera">
+		<visual>
+			<origin xyz="-0.0 0 0.05" rpy="0 -1.5707 1.5707" />
 			<geometry>
 				<mesh filename="package://robot/meshes/kinect.dae" />
@@ -190,9 +215,8 @@
 		</inertial>
 	</link>
-	<joint type="fixed" name="camera_joint">
-		<origin xyz="0.4 0 0" rpy="0 0 0" />
-		<child link="camera" />
-		<parent link="chassis" />
-		<axis xyz="0 1 0" rpy="0 0 0" />
+	<joint type="fixed" name="RGBD_camera_joint">
+		<origin xyz="0.0 0 0.0" rpy="-1.5707 0 -1.5707" />
+		<child link="RGBD_camera" />
+		<parent link="camera" />
 	</joint>
 	<!-- LIDAR -->
